File: Optimus/Hardware/shield passage vitesse.sch (EAGLE design)
At the start: 37 parts, among them Q1 2N7000, Q2 2N7000, Q3 2N7000, Q4 2N7000, Q5 2N7000

Commit message: Passage de la Zener à 15V et ajout des convention +5 V et +12V
Parts:
- C4, C5: value 0.33uF -> 0.33µF
- D1: value ZENER 12V -> ZENER 15V
- F1: value 1A -> 2A
Connections:
- net 12V renamed +12V
- net 5V renamed +5V
